Commit message: initial fork

File: bluerov2_description/robots/bluerov2_default.xacro (robot description, xacro)
@@ -3,4 +3,5 @@
   <xacro:arg name="debug" default="0"/>
   <xacro:arg name="namespace" default="bluerov2"/>
+  <!--<xacro:arg name="inertial_reference_frame" default="world"/>-->
   <!-- Include the ROV macro file xacro:bluerov2_base -->
   <xacro:include filename="$(find bluerov2_description)/urdf/base.xacro"/>
@@ -8,9 +9,11 @@
   <xacro:include filename="$(find bluerov2_description)/urdf/gazebo.xacro"/>
 <!-- Create the bluerov2 -->
-  <xacro:bluerov2_base namespace="$(arg namespace)">
+  <xacro:bluerov2_base
+    namespace="$(arg namespace)">
+    <!--inertial_reference_frame="$(arg inertial_reference_frame)">-->
     <!-- The underwater object plugin is given as an input block parameter to
      allow the addition of external models of manipulator units -->
     <gazebo>
-      <plugin name="uuv_plugin" filename="libunderwater_object_ros_plugin.so">
+      <plugin name="uuv_plugin" filename="libuuv_underwater_object_ros_plugin.so">
         <fluid_density>1028.0</fluid_density>
         <flow_velocity_topic>hydrodynamics/current_velocity</flow_velocity_topic>

File: bluerov2_description/urdf/actuators.xacro (robot description, xacro)
@@ -8,26 +8,46 @@
     aware that Gazebo does not use the SNAME convention per default.
   -->
+ <gazebo>
+   <plugin name="gazebo_ros_control" filename="libgazebo_ros_control.so">
+     <robotNamespace>/$(arg namespace)</robotNamespace>
+     <robotParam>/$(arg namespace)/robot_description</robotParam>
+   </plugin>
+ </gazebo>
+  <xacro:include filename="$(find uuv_gazebo_ros_plugins)/urdf/thruster_snippets.xacro"/>
+  <xacro:property name="prop_mesh_file" value="file://$(find bluerov2_description)/meshes/bluerov2_propcw.dae"/>
+  <!-- Thruster joint and link snippet -->
+  <xacro:macro name="thruster_macro"
+    params="namespace thruster_id *origin">
+    <xacro:thruster_module_first_order_basic_fcn_macro
+      namespace="${namespace}"
+      thruster_id="${thruster_id}"
+      mesh_filename="${prop_mesh_file}"
+      dyn_time_constant="0.05"
+      rotor_constant="0.1">
+      <xacro:insert_block name="origin"/>
+    </xacro:thruster_module_first_order_basic_fcn_macro>
+  </xacro:macro>
   <!-- IMPROVE -->
-  <xacro:thruster_macro robot_namespace="${namespace}" thruster_id="0">
+  <xacro:thruster_macro namespace="${namespace}" thruster_id="0">
     <origin xyz="0.1355 -0.1 -0.0725" rpy="0 0 0.7853981634"/>
   </xacro:thruster_macro>
   <!-- IMPROVE -->
-  <xacro:thruster_macro robot_namespace="${namespace}" thruster_id="1">
+  <xacro:thruster_macro namespace="${namespace}" thruster_id="1">
     <origin xyz="0.1355 0.1 -0.0725" rpy="0 0 -0.7853981634"/>
   </xacro:thruster_macro>
   <!-- IMPROVE -->
-  <xacro:thruster_macro robot_namespace="${namespace}" thruster_id="2">
+  <xacro:thruster_macro namespace="${namespace}" thruster_id="2">
     <origin xyz="-0.1475 -0.1 -0.0725" rpy="0 0 2.3561944902"/>
   </xacro:thruster_macro>
   <!-- IMPROVE -->
-  <xacro:thruster_macro robot_namespace="${namespace}" thruster_id="3">
+  <xacro:thruster_macro namespace="${namespace}" thruster_id="3">
     <origin xyz="-0.1475 0.1 -0.0725" rpy="0 0 -2.3561944902"/>
   </xacro:thruster_macro>
   <!-- IMPROVE -->
-  <xacro:thruster_macro robot_namespace="${namespace}" thruster_id="4">
+  <xacro:thruster_macro namespace="${namespace}" thruster_id="4">
     <origin xyz="0.0025 -0.1105 -0.005" rpy="0 -1.5707963268 0"/>
   </xacro:thruster_macro>
   <!-- IMPROVE -->
-  <xacro:thruster_macro robot_namespace="${namespace}" thruster_id="5">
+  <xacro:thruster_macro namespace="${namespace}" thruster_id="5">
     <origin xyz="0.0025 0.1105 -0.005" rpy="0 -1.5707963268 0"/>
   </xacro:thruster_macro>

File: bluerov2_description/urdf/base.xacro (robot description, xacro)
@@ -2,7 +2,8 @@
 <robot xmlns:xacro="http://www.ros.org/wiki/xacro">
   <!-- Loading some constants -->
-  <xacro:include filename="$(find uuv_descriptions)/models/common/urdf/common.urdf.xacro"/>
+  <xacro:include filename="$(find uuv_descriptions)/urdf/common.urdf.xacro"/>
   <!-- Loading file with sensor macros -->
   <xacro:include filename="$(find uuv_sensor_ros_plugins)/urdf/sensor_snippets.xacro"/>
+  <xacro:include filename="$(find uuv_gazebo_ros_plugins)/urdf/snippets.xacro"/>
   <!-- Loading vehicle's specific macros -->
   <xacro:include filename="$(find bluerov2_description)/urdf/snippets.xacro"/>
@@ -20,5 +21,5 @@
   <!-- minion_usv_height is not really! It's just for run... We need first calculate the Fossen parameters -->
   <!-- Volume -->
-  <xacro:property name="volume" value="0.011054"/>
+  <xacro:property name="volume" value="0.0299753"/>
   <!-- Center of gravity -->
   <xacro:property name="cog" value="0 0 0"/>
@@ -72,9 +73,29 @@
         </visual>
         <!-- In rexrov2_base they made collision planes to minize the GPU load -->
-        <!-- <collision>
+        <collision>
           <origin xyz="0 0 0" rpy="0 0 0"/>
           <geometry>
             <mesh filename="${collision_mesh_file}" scale="1 1 1" />
           </geometry>
+        </collision>
+        <!-- <collision>
+          <origin xyz="0 0 -0.75" rpy="0 0 0"/>
+          <geometry>
+           <box size="2.56 1.50 0.10"/>
+          </geometry>
+        </collision> -->
+        <!-- top plate -->
+        <!-- <collision>
+          <origin xyz="0 0 0.60" rpy="0 0 0"/>
+          <geometry><box size="2.56 1.50 0.40"/></geometry>
+        </collision> -->
+        <!-- left / right sides -->
+        <!-- <collision>
+          <origin xyz="-0.20 0.70 -0.15" rpy="0 0 0"/>
+          <geometry><box size="2.20 0.10 1.10"/></geometry>
+        </collision>
+        <collision>
+           <origin xyz="-0.20 -0.70 -0.15" rpy="0 0 0"/>
+           <geometry><box size="2.20 0.10 1.10"/></geometry>
         </collision> -->
       </link>

File: bluerov2_description/urdf/gazebo.xacro (robot description, xacro)
@@ -5,5 +5,5 @@
     <link name="${namespace}/base_link">
       <!-- This flag will make the link neutrally buoyant -->
-      <neutrally_buoyant>0</neutrally_buoyant>
+      <neutrally_buoyant>1</neutrally_buoyant>
       <!-- Link's volume -->
       <volume>${volume}</volume>
@@ -27,10 +27,28 @@
           <!-- Added mass: see p.28 in Berg2012 -->
           <added_mass>
-            1.7182 0 0 0 0 0
+            <!-- 779.79 -6.8773 -103.32  8.5426 -165.54 -7.8033
+           -6.8773    1222   51.29  409.44 -5.8488  62.726
+           -103.32   51.29  3659.9  6.1112 -386.42  10.774
+           8.5426  409.44  6.1112   534.9 -10.027  21.019
+           -165.54 -5.8488 -386.42 -10.027  842.69 -1.1162
+           -7.8033  62.726  10.775  21.019 -1.1162  224.32 -->
+            <!-- 1.7182 0 0 0 0 0
             0 0 0 0 0 0
             0 0 5.468 0 0 0
             0 0 0 0 0 0
             0 0 0 0 1.2481 0
-            0 0 0 0 0 0.4006
+            0 0 0 0 0 0.4006 -->
+            <!-- 20 0 0 0 0 0
+            0 20 0 0 0 0
+            0 0 20 0 0 0
+            0 0 0 30 0 0
+            0 0 0 0 30 0
+            0 0 0 0 0 30 -->
+            11.985 -0.091 -0.105 0.039 0.308 0.012
+            0.149 20.261 -0.147 0.085 -0.013 -0.785
+            0.111 -0.129 67.141 -0.033 2.530 0.064
+            0.122 0.319 -0.056 0.385 0.003 -0.011
+            0.407 -0.001 2.543 -0.002 0.791 0.002
+            -0.003 -0.758 0.064 -0.003 -0.004 0.138
           </added_mass>
           <!--
@@ -40,5 +58,7 @@
           -->
           <linear_damping>
+            <!-- -74.82 -69.48 -728.4 -268.8 -309.77 -105 -->
             -11.7391 -20 -31.8678 -25 -44.9085 -5
+            <!-- -20.63 -54.03 -61.05 -50 -50 -26.90-->
           </linear_damping>
           <!--
@@ -48,7 +68,7 @@
             This matrix is mostly useful for slender bodies (e.g. AUVs with torpedo shape)
           -->
-          <!-- <linear_damping_forward_speed>
+          <linear_damping_forward_speed>
             0 0 0 0 0 0
-          </linear_damping_forward_speed> -->
+          </linear_damping_forward_speed>
           <!--
             The quadratic damping coefficients can be provided as a diagonal (6 elements)
@@ -57,5 +77,6 @@
           -->
           <quadratic_damping>
-            0 0 0 0 0 0
+            -748.22 -992.53 -1821.01 -672 -774.44 -523.27
+            <!-- -151.83 -270.15 -176.54 -200 -200 -17.52 -->
           </quadratic_damping>
           <!--

File: bluerov2_description/urdf/sensors.xacro (robot description, xacro)
@@ -8,20 +8,27 @@
   -->
   <!-- Mount a Pose 3D sensor. -->
-  <xacro:default_pose_3d namespace="${namespace}" parent_link="${namespace}/base_link" />
+  <!--<xacro:default_pose_3d namespace="${namespace}" parent_link="${namespace}/base_link" />-->
+  <xacro:include filename="$(find uuv_gazebo_ros_plugins)/urdf/snippets.xacro"/>
   <!-- IMU Sensor -->
-  <xacro:default_imu namespace="${namespace}" parent_link="${namespace}/base_link">
+  <xacro:default_imu_macro
+    namespace="${namespace}"
+    parent_link="${namespace}/base_link"
+    inertial_reference_frame="world">
     <origin xyz="0 0 0" rpy="0 0 0"/>
-  </xacro:default_imu>
+  </xacro:default_imu_macro>
   <!-- Pressure Sensor  -->
   <xacro:default_pressure namespace="${namespace}" parent_link="${namespace}/base_link">
     <origin xyz="0 0 0" rpy="0 0 0"/>
   </xacro:default_pressure>
-  <!-- Beacon Sensor  -->
+  <!-- Beacon Sensor
   <xacro:default_beacon namespace="${namespace}" parent_link="${namespace}/base_link">
     <origin xyz="0 0 0" rpy="0 0 0"/>
-  </xacro:default_beacon>
+  </xacro:default_beacon> -->
   <!-- Mount a camera -->
-  <!-- <xacro:default_camera namespace="${namespace}" parent_link="${namespace}/base_link" suffix="front">
-    <origin xyz="0 0 0.2" rpy="0 0 0"/>
-  </xacro:default_camera> -->
+  <xacro:default_camera namespace="${namespace}" parent_link="${namespace}/base_link" suffix="right">
+    <origin xyz=".23 -0.18 0.03" rpy="0 0.4 0.0"/>
+  </xacro:default_camera>
+  <xacro:default_camera namespace="${namespace}" parent_link="${namespace}/base_link" suffix="left">
+    <origin xyz=".23 0.18 0.03" rpy="0 0.4 -0.0"/>
+  </xacro:default_camera>
 </robot>

File: bluerov2_description/urdf/snippets.xacro (robot description, xacro)
@@ -10,5 +10,5 @@
     be initialized in the actuators.xacro file.
   -->
-  <xacro:macro name="thruster_macro" params="robot_namespace thruster_id *origin">
+  <!-- <xacro:macro name="thruster_macro" params="robot_namespace thruster_id *origin"> -->
     <!--
     Dummy link as place holder for the thruster frame,
@@ -16,5 +16,5 @@
     of the vehicle and may cause internal collisions if set otherwise
     -->
-    <link name="${robot_namespace}/thruster_${thruster_id}">
+   <!--  <link name="${robot_namespace}/thruster_${thruster_id}">
       <visual>
         <geometry>
@@ -29,24 +29,24 @@
                izz="0.000000017" />
       </inertial>
-    </link>
+    </link> -->
     <!-- Joint between thruster link and vehicle base link -->
-    <joint name="${robot_namespace}/thruster_${thruster_id}_joint" type="continuous">
+    <!-- <joint name="${robot_namespace}/thruster_${thruster_id}_joint" type="continuous">
       <xacro:insert_block name="origin" />
       <axis xyz="1 0 0" />
       <parent link="${robot_namespace}/base_link" />
       <child link="${robot_namespace}/thruster_${thruster_id}" />
-    </joint>
-    <!-- From desistek underwater vehicle -->
-    <gazebo>
+    </joint> -->
+    <!-- From desistek underwater vehicle
+    <gazebo> -->
       <!-- Thruster ROS plugin -->
-     <plugin name="${robot_namespace}_${thruster_id}_thruster_model" filename="libthruster_ros_plugin.so">
+     <!-- <plugin name="${robot_namespace}_${thruster_id}_thruster_model" filename="libthruster_ros_plugin.so"> -->
        <!-- Name of the thruster link -->
-       <linkName>${robot_namespace}/thruster_${thruster_id}</linkName>
+       <!-- <linkName>${robot_namespace}/thruster_${thruster_id}</linkName> -->
        <!-- Name of the joint between thruster and vehicle base link -->
-       <jointName>${robot_namespace}/thruster_${thruster_id}_joint</jointName>
+       <!-- <jointName>${robot_namespace}/thruster_${thruster_id}_joint</jointName> -->
        <!-- Make the thruster aware of its id -->
-       <thrusterID>${thruster_id}</thrusterID>
+       <!-- <thrusterID>${thruster_id}</thrusterID> -->
        <!-- Gain of the input command signal -->
-       <gain>1</gain>
+       <!-- <gain>1</gain> -->
        <!-- Maximum allowed input value for the input signal for thruster unit -->
        <!-- <clampMax>0</clampMax> -->
@@ -60,5 +60,5 @@
        Default value is 1.0
        -->
-       <thrust_efficiency>1</thrust_efficiency>
+       <!-- <thrust_efficiency>1</thrust_efficiency> -->
        <!--
        Value from 0 to 1 to set the efficiency of the propeller as a factor
@@ -67,7 +67,7 @@
        Default value is 1.0
        -->
-       <propeller_efficiency>1</propeller_efficiency>
+       <!-- <propeller_efficiency>1</propeller_efficiency> -->
        <!-- 2) First order model -->
-       <dynamics>
+       <!-- <dynamics>
          <type>FirstOrder</type>
          <timeConstant>0.2</timeConstant>
@@ -75,7 +75,7 @@
        <conversion>
          <type>Basic</type>
-         <rotorConstant>0.00001</rotorConstant>
+         <rotorConstant>0.00001</rotorConstant> -->
          <!-- <rotorConstant>0</rotorConstant> -->
-       </conversion>
+       <!-- </conversion>
      </plugin>
    </gazebo>
@@ -83,4 +83,4 @@
       <selfCollide>false</selfCollide>
     </gazebo>
-  </xacro:macro>
+  </xacro:macro> -->
 </robot>
