Commit message: as of 7/18

File: bluerov2_description/urdf/base.xacro (robot description, xacro)
@@ -73,30 +73,30 @@
         </visual>
         <!-- In rexrov2_base they made collision planes to minize the GPU load -->
-        <collision>
+        <!--<collision>
           <origin xyz="0 0 0" rpy="0 0 0"/>
           <geometry>
             <mesh filename="${collision_mesh_file}" scale="1 1 1" />
           </geometry>
+        </collision>-->
+        <collision>
+          <origin xyz="0 0 -0.14033" rpy="0 0 0"/>
+          <geometry>
+           <box size="0.448 0.2384 0.010"/>
+          </geometry>
         </collision>
-        <!-- <collision>
-          <origin xyz="0 0 -0.75" rpy="0 0 0"/>
-          <geometry>
-           <box size="2.56 1.50 0.10"/>
-          </geometry>
-        </collision> -->
         <!-- top plate -->
-        <!-- <collision>
-          <origin xyz="0 0 0.60" rpy="0 0 0"/>
-          <geometry><box size="2.56 1.50 0.40"/></geometry>
-        </collision> -->
+        <collision>
+          <origin xyz="0 0 0.14033" rpy="0 0 0"/>
+          <geometry><box size="0.448 0.2384 0.010"/></geometry>
+        </collision>
         <!-- left / right sides -->
-        <!-- <collision>
-          <origin xyz="-0.20 0.70 -0.15" rpy="0 0 0"/>
-          <geometry><box size="2.20 0.10 1.10"/></geometry>
+        <collision>
+          <origin xyz="-0 0.1192 0" rpy="0 0 0"/>
+          <geometry><box size="0.448 0.010 0.28066"/></geometry>
         </collision>
         <collision>
-           <origin xyz="-0.20 -0.70 -0.15" rpy="0 0 0"/>
-           <geometry><box size="2.20 0.10 1.10"/></geometry>
-        </collision> -->
+           <origin xyz="-0 -0.1192 0" rpy="0 0 0"/>
+           <geometry><box size="0.448 0.010 0.28066"/></geometry>
+        </collision>
       </link>
     <gazebo reference="${namespace}/base_link">

File: bluerov2_description/urdf/gazebo.xacro (robot description, xacro)
@@ -45,10 +45,16 @@
             0 0 0 0 30 0
             0 0 0 0 0 30 -->
-            11.985 -0.091 -0.105 0.039 0.308 0.012
+            <!--11.985 -0.091 -0.105 0.039 0.308 0.012
             0.149 20.261 -0.147 0.085 -0.013 -0.785
             0.111 -0.129 67.141 -0.033 2.530 0.064
             0.122 0.319 -0.056 0.385 0.003 -0.011
             0.407 -0.001 2.543 -0.002 0.791 0.002
-            -0.003 -0.758 0.064 -0.003 -0.004 0.138
+            -0.003 -0.758 0.064 -0.003 -0.004 0.138-->
+            18.814 0 0 0 0 0
+            0 30.1 0 0 0 0
+            0 0 30.1 0 0 0
+            0 0 0 0.113 0 0
+            0 0 0 0 0.1726 0
+            0 0 0 0 0 0.2429
           </added_mass>
           <!--
@@ -59,5 +65,6 @@
           <linear_damping>
             <!-- -74.82 -69.48 -728.4 -268.8 -309.77 -105 -->
-            -11.7391 -20 -31.8678 -25 -44.9085 -5
+            <!-- -11.7391 -20 -31.8678 -25 -44.9085 -5-->
+            -8.814 -20.1 -20.1 0 .0604 -.0279
             <!-- -20.63 -54.03 -61.05 -50 -50 -26.90-->
           </linear_damping>
@@ -77,5 +84,6 @@
           -->
           <quadratic_damping>
-            -748.22 -992.53 -1821.01 -672 -774.44 -523.27
+            <!-- -748.22 -992.53 -1821.01 -672 -774.44 -523.27-->
+            -21.42 -28.41 -52.13 -19.24 -22.17 -14.98
             <!-- -151.83 -270.15 -176.54 -200 -200 -17.52 -->
           </quadratic_damping>

File: bluerov2_description/urdf/sensors.xacro (robot description, xacro)
@@ -32,3 +32,10 @@
     <origin xyz=".23 0.18 0.03" rpy="0 0.4 -0.0"/>
   </xacro:default_camera>
+  <!-- for balance -->
+  <xacro:default_camera namespace="${namespace}" parent_link="${namespace}/base_link" suffix="backright">
+    <origin xyz="-.23 -0.18 0.03" rpy="0 0.4 0.0"/>
+  </xacro:default_camera>
+  <xacro:default_camera namespace="${namespace}" parent_link="${namespace}/base_link" suffix="backleft">
+    <origin xyz="-.23 0.18 0.03" rpy="0 0.4 -0.0"/>
+  </xacro:default_camera>
 </robot>
