Commit message: Update actuators.xacro

File: bluerov2_description/urdf/actuators.xacro (robot description, xacro)
@@ -30,9 +30,9 @@
   <!-- IMPROVE -->
   <xacro:thruster_macro namespace="${namespace}" thruster_id="0">
-    <origin xyz="0.1355 -0.1 -0.0725" rpy="0 0 0.7853981634"/>
+    <origin xyz="0.1475 -0.1 -0.0725" rpy="0 0 0.7853981634"/>
   </xacro:thruster_macro>
   <!-- IMPROVE -->
   <xacro:thruster_macro namespace="${namespace}" thruster_id="1">
-    <origin xyz="0.1355 0.1 -0.0725" rpy="0 0 -0.7853981634"/>
+    <origin xyz="0.1475 0.1 -0.0725" rpy="0 0 -0.7853981634"/>
   </xacro:thruster_macro>
   <!-- IMPROVE -->
@@ -46,9 +46,9 @@
   <!-- IMPROVE -->
   <xacro:thruster_macro namespace="${namespace}" thruster_id="4">
-    <origin xyz="0.0025 -0.1105 -0.005" rpy="0 -1.5707963268 0"/>
+    <origin xyz="0 -0.1105 -0.005" rpy="0 -1.5707963268 0"/>
   </xacro:thruster_macro>
   <!-- IMPROVE -->
   <xacro:thruster_macro namespace="${namespace}" thruster_id="5">
-    <origin xyz="0.0025 0.1105 -0.005" rpy="0 -1.5707963268 0"/>
+    <origin xyz="0 0.1105 -0.005" rpy="0 -1.5707963268 0"/>
   </xacro:thruster_macro>
   <!-- ###### TO BE IMPLEMENTED ###### -->

Commit message: 9-21 update

File: bluerov2_description/urdf/actuators.xacro (robot description, xacro)
@@ -28,27 +28,27 @@
     </xacro:thruster_module_first_order_basic_fcn_macro>
   </xacro:macro>
-  <!-- IMPROVE -->
+  <!-- IMPROVE Front left-->
   <xacro:thruster_macro namespace="${namespace}" thruster_id="0">
-    <origin xyz="0.1475 -0.1 -0.0725" rpy="0 0 0.7853981634"/>
+    <origin xyz="0.1475 -0.1 -0.0" rpy="0 0 0.7853981634"/>
   </xacro:thruster_macro>
-  <!-- IMPROVE -->
+  <!-- IMPROVE front right-->
   <xacro:thruster_macro namespace="${namespace}" thruster_id="1">
-    <origin xyz="0.1475 0.1 -0.0725" rpy="0 0 -0.7853981634"/>
+    <origin xyz="0.1475 0.1 -0.0" rpy="0 0 -0.7853981634"/>
   </xacro:thruster_macro>
-  <!-- IMPROVE -->
+  <!-- IMPROVE back left-->
   <xacro:thruster_macro namespace="${namespace}" thruster_id="2">
-    <origin xyz="-0.1475 -0.1 -0.0725" rpy="0 0 2.3561944902"/>
+    <origin xyz="-0.1475 -0.1 -0.0" rpy="0 0 2.3561944902"/>
   </xacro:thruster_macro>
-  <!-- IMPROVE -->
+  <!-- IMPROVE back right-->
   <xacro:thruster_macro namespace="${namespace}" thruster_id="3">
-    <origin xyz="-0.1475 0.1 -0.0725" rpy="0 0 -2.3561944902"/>
+    <origin xyz="-0.1475 0.1 -0.0" rpy="0 0 -2.3561944902"/>
   </xacro:thruster_macro>
-  <!-- IMPROVE -->
+  <!-- IMPROVE left-->
   <xacro:thruster_macro namespace="${namespace}" thruster_id="4">
-    <origin xyz="0 -0.1105 -0.005" rpy="0 -1.5707963268 0"/>
+    <origin xyz="0.00 -0.1105 -0.005" rpy="0 -1.5707963268 0"/>
   </xacro:thruster_macro>
-  <!-- IMPROVE -->
+  <!-- IMPROVE right-->
   <xacro:thruster_macro namespace="${namespace}" thruster_id="5">
-    <origin xyz="0 0.1105 -0.005" rpy="0 -1.5707963268 0"/>
+    <origin xyz="0.00 0.1105 -0.005" rpy="0 -1.5707963268 0"/>
   </xacro:thruster_macro>
   <!-- ###### TO BE IMPLEMENTED ###### -->

File: bluerov2_description/urdf/base.xacro (robot description, xacro)
@@ -29,5 +29,5 @@
   assume NWU (otherwise cob is below cog?). 0.155
   -->
-  <xacro:property name="cob" value="0 0 0"/>
+  <xacro:property name="cob" value="0 0 .16"/>
   <!-- Fluid density -->
   <xacro:property name="rho" value="1028"/>
@@ -101,4 +101,40 @@
       </link>
     <gazebo reference="${namespace}/base_link">
+      <light type="spot" name="light1">
+        <cast_shadows>0</cast_shadows>
+        <pose>.23 0.18 0.03 0 -1.5707 -0.0</pose>
+        <diffuse>1 1 1 1</diffuse>
+        <specular>1 1 1 1</specular>
+        <intensity>10</intensity>
+        <attenuation>
+          <range>20.0</range>
+          <constant>0.0</constant>
+          <linear>.03</linear>
+        </attenuation>
+        <spot>
+          <inner_angle>2.356</inner_angle>
+          <outer_angle>3.1415</outer_angle>
+          <falloff>1</falloff>
+        </spot>
+        <direction>0 0 -1</direction>
+      </light>
+      <light type="spot" name="light2">
+        <cast_shadows>0</cast_shadows>
+        <pose>.23 -0.18 0.03 0 -1.5707 -0.0</pose>
+        <diffuse>1 1 1 1</diffuse>
+        <specular>1 1 1 1</specular>
+        <intensity>10</intensity>
+        <attenuation>
+          <range>20.0</range>
+          <constant>0.0</constant>
+          <linear>.03</linear>
+        </attenuation>
+        <spot>
+          <inner_angle>2.356</inner_angle>
+          <outer_angle>3.1415</outer_angle>
+          <falloff>1</falloff>
+        </spot>
+        <direction>0 0 -1</direction>
+      </light>
       <selfCollide>false</selfCollide>
     </gazebo>

File: bluerov2_description/urdf/sensors.xacro (robot description, xacro)
@@ -8,5 +8,5 @@
   -->
   <!-- Mount a Pose 3D sensor. -->
-  <!--<xacro:default_pose_3d namespace="${namespace}" parent_link="${namespace}/base_link" />-->
+  <xacro:default_pose_3d namespace="${namespace}" parent_link="${namespace}/base_link" />
   <xacro:include filename="$(find uuv_gazebo_ros_plugins)/urdf/snippets.xacro"/>
   <!-- IMU Sensor -->
@@ -39,3 +39,6 @@
     <origin xyz="-.23 0.18 0.03" rpy="0 0.4 -0.0"/>
   </xacro:default_camera>
+  <!--<xacro:light_link_macro namespace="${namespace}" parent_link="${namespace}/base_link" suffix="1">
+    <origin xyz=".23 -0.18 0.03" rpy="0 0 0"/>
+  </xacro:light_link_macro>-->
 </robot>
